File: kicad/smart-psu.sch (KiCad schematic (older format))
At the start: 13 parts, among them J1 12V, Q1 AOD4184A, U1 LM2596, U2 ATTINY13-20SSU

Commit message: Power switch on INT0
Connections:
- wire segments 36 -> 46
Changed lines of the file:
@@
 	3350 3750 3300 3750
 Wire Wire Line
-	3300 3550 3650 3550
+	3300 3550 3600 3550
+Wire Wire Line
+	3600 3550 3650 3550
 Wire Wire Line
 	5200 3750 5150 3750
 Wire Wire Line
-	4850 3750 4950 3750
+	4850 3750 4900 3750
 Wire Wire Line
-	5600 3400 5600 3800
+	4900 3750 4950 3750
+Wire Wire Line
+	5600 3400 5600 3550
+Wire Wire Line
+	5600 3550 5600 3800
 $Comp
 L 2N7002 Q1
@@
 $EndComp
 Wire Wire Line
-	5200 3000 5200 3800
+	5200 3000 5200 3550
+Wire Wire Line
+	5200 3550 5200 3750
+Wire Wire Line
+	5200 3750 5200 3800
 $Comp
 L GND #PWR015
@@
 $EndComp
 Wire Wire Line
-	7900 3050 8150 3050
+	7900 3050 8050 3050
+Wire Wire Line
+	8050 3050 8150 3050
 Connection ~ 8050 3050
 Wire Wire Line
-	4850 3550 5300 3550
+	4850 3550 5200 3550
 Wire Wire Line
-	5500 3550 6100 3550
+	5200 3550 5300 3550
 Wire Wire Line
-	8050 3350 8800 3350
+	5500 3550 5600 3550
+Wire Wire Line
+	5600 3550 5800 3550
+Wire Wire Line
+	5800 3550 6100 3550
+Wire Wire Line
+	8050 3350 8350 3350
+Wire Wire Line
+	8350 3350 8800 3350
 Wire Wire Line
 	8050 3350 8050 3300

Commit message: Update schematic for high-side switch.
Parts:
- removed Q1: AOD4184A, TO_SOT_Packages_SMD:SOT-23, symbol 2N7002
- removed R1: 4k7, Resistors_SMD:R_1206_HandSoldering, symbol R_Small
- added D3: PWR, symbol LED_Small_ALT
- added J2: Conn_01x05, symbol Conn_01x05
- added Q1: P2003ED, symbol Q_PMOS_GDS
- added Q2: TUP, symbol Q_NPN_BEC
- added R2: 470R, symbol R_Small
- added R3: 2k2, symbol R_Small
- added R?: 10k, symbol R_Small
- added SW1: SW_DIP_x02, Buttons_Switches_THT:SW_DIP_x2_Slide, symbol SW_DIP_x02
- added U3: AZ1117-3.3, Diodes_SMD:D_SOD-123, symbol AZ1117-3.3
- C3: value 100u -> 10u
Connections:
- net labels added: DELAY1, DELAY2, ~HB
- net labels removed: DELAY, LED
- wire segments 46 -> 57
- no-connect marks 1 -> 0

Commit message: Upgrade to Kicad 5.0
Parts:
- C1, C2, C3: symbol CP1_Small -> Device:CP1_Small
- C4: symbol C_Small -> Device:C_Small
- D1, D2: symbol D_Schottky_Small_ALT -> smart-psu-rescue:D_Schottky_Small_ALT
- D3: symbol LED_Small_ALT -> Device:LED_Small_ALT
- F1: symbol Fuse_Small -> Device:Fuse_Small
- J1: symbol Screw_Terminal_1x02 -> smart-psu-rescue:Screw_Terminal_1x02
- J2: symbol Conn_01x05 -> smart-psu-rescue:Conn_01x05
- L1: symbol L_Core_Ferrite_Small -> Device:L_Core_Ferrite_Small
- Q1: symbol Q_PMOS_GDS -> Device:Q_PMOS_GDS
- Q2: symbol Q_NPN_BEC -> Device:Q_NPN_BEC
- R2, R3, R?: symbol R_Small -> Device:R_Small
- SW1: symbol SW_DIP_x02 -> smart-psu-rescue:SW_DIP_x02
- U1: symbol LM2596 -> smart-psu-rescue:LM2596
- U2: symbol ATTINY13-20SSU -> smart-psu-rescue:ATTINY13-20SSU
- U3: symbol AZ1117-3.3 -> smart-psu-rescue:AZ1117-3.3
Connections:
- wire segments 57 -> 69
Changed lines of the file:
@@
-EESchema Schematic File Version 2
-LIBS:power
-LIBS:device
-LIBS:transistors
-LIBS:conn
-LIBS:regul
+EESchema Schematic File Version 4
 LIBS:smart-psu-cache
-EELAYER 25 0
+EELAYER 26 0
 EELAYER END
 $Descr A4 11693 8268
@@
 $EndDescr
 $Comp
-L C_Small C4
+L Device:C_Small C4
 U 1 1 5A367225
 P 5800 3900
@@
 ~PWRON
 $Comp
-L GND #PWR11
+L power:GND #PWR11
 U 1 1 5A36723C
 P 5100 4050
@@
 $EndComp
 $Comp
-L PWR_FLAG #FLG2
+L power:PWR_FLAG #FLG2
 U 1 1 5A36723E
 P 3400 4950
@@
 $EndComp
 $Comp
-L PWR_FLAG #FLG1
+L power:PWR_FLAG #FLG1
 U 1 1 5A36723F
 P 3000 5200
@@
 $EndComp
 $Comp
-L GND #PWR4
+L power:GND #PWR4
 U 1 1 5A367240
 P 3400 5200
@@
 $EndComp
 $Comp
-L +5V #PWR2
+L power:+5V #PWR2
 U 1 1 5A367241
 P 3000 4950
@@
 $EndComp
 $Comp
-L ATTINY13-20SSU U2
+L smart-psu-rescue:ATTINY13-20SSU U2
 U 1 1 5A36742E
 P 7050 3800
@@
 $EndComp
 $Comp
-L GND #PWR15
+L power:GND #PWR15
 U 1 1 5A367BD2
 P 6000 4250
@@
 $EndComp
 Wire Wire Line
-	5800 3350 5800 3800
+	5800 3350 5800 3550
 Connection ~ 5800 3550
 $Comp
-L LM2596 U1
+L smart-psu-rescue:LM2596 U1
 U 1 1 5A37884F
 P 3850 3650
@@
 $EndComp
 $Comp
-L GND #PWR5
+L power:GND #PWR5
 U 1 1 5A378850
 P 3700 4050
@@
 $EndComp
 $Comp
-L GND #PWR7
+L power:GND #PWR7
 U 1 1 5A378851
 P 4000 4050
@@
 	4000 4050 4000 4000
 $Comp
-L L_Core_Ferrite_Small L1
+L Device:L_Core_Ferrite_Small L1
 U 1 1 5A378852
 P 4650 3750
@@
 $EndComp
 $Comp
-L D_Schottky_Small_ALT D1
+L smart-psu-rescue:D_Schottky_Small_ALT D1
 U 1 1 5A378853
 P 4500 3900
@@
 Connection ~ 4500 3750
 $Comp
-L GND #PWR8
+L power:GND #PWR8
 U 1 1 5A378854
 P 4500 4050
@@
 	4500 4050 4500 4000
 $Comp
-L CP1_Small C2
+L Device:CP1_Small C2
 U 1 1 5A378855
 P 4800 3900
@@
 $EndComp
 $Comp
-L GND #PWR10
+L power:GND #PWR10
 U 1 1 5A378856
 P 4800 4050
@@
 	4800 4050 4800 4000
 $Comp
-L +5V #PWR9
+L power:+5V #PWR9
 U 1 1 5A378857
 P 4800 3000
@@
 Connection ~ 4800 3550
 $Comp
-L CP1_Small C1
+L Device:CP1_Small C1
 U 1 1 5A378858
 P 3200 3900
@@
 $EndComp
 $Comp
-L GND #PWR3
+L power:GND #PWR3
 U 1 1 5A378859
 P 3200 4050
@@
 Connection ~ 3200 3550
 $Comp
-L Screw_Terminal_1x02 J1
+L smart-psu-rescue:Screw_Terminal_1x02 J1
 U 1 1 5A37885A
 P 2750 3650
@@
 $EndComp
 $Comp
-L GND #PWR1
+L power:GND #PWR1
 U 1 1 5A37885B
 P 3000 4050
@@
 	4800 3750 4750 3750
 Wire Wire Line
-	4450 3750 4550 3750
-$Comp
-L +5V #PWR16
+	4450 3750 4500 3750
+$Comp
+L power:+5V #PWR16
 U 1 1 5A3824C8
 P 6550 2050
@@
 $EndComp
 Wire Wire Line
-	4800 3000 4800 3800
-$Comp
-L GND #PWR14
+	4800 3000 4800 3550
+$Comp
+L power:GND #PWR14
 U 1 1 5A3827DD
 P 5800 4050
@@
 	3400 5200 3400 4950
 $Comp
-L D_Schottky_Small_ALT D2
+L smart-psu-rescue:D_Schottky_Small_ALT D2
 U 1 1 5A382D9D
 P 4950 3550
@@
 $EndComp
 $Comp
-L Fuse_Small F1
+L Device:Fuse_Small F1
 U 1 1 5A38D757
 P 6700 2100
@@
 ~PWRON
 $Comp
-L VCC #PWR13
+L power:VCC #PWR13
 U 1 1 5A79EF6A
 P 5800 3350
@@
 $EndComp
 $Comp
-L VCC #PWR6
+L power:VCC #PWR6
 U 1 1 5A79F05F
 P 3800 4950
@@
 $EndComp
 $Comp
-L PWR_FLAG #FLG3
+L power:PWR_FLAG #FLG3
 U 1 1 5A79F091
 P 3800 5200
@@
 	6000 4050 6050 4050
 $Comp
-L GND #PWR19
+L power:GND #PWR19
 U 1 1 5AB88D16
 P 8950 4150
@@
 	9050 3550 8750 3550
 $Comp
-L LED_Small_ALT D3
+L Device:LED_Small_ALT D3
 U 1 1 5AC21F2C
 P 7500 2700
@@
 $EndComp
 $Comp
-L GND #PWR18
+L power:GND #PWR18
 U 1 1 5ACA4675
 P 7500 2950
@@
 DELAY1
 $Comp
-L R_Small R2
+L Device:R_Small R2
 U 1 1 5AC2239F
 P 7500 2300
@@
 LOAD
 $Comp
-L R_Small R3
+L Device:R_Small R3
 U 1 1 5ACA818F
 P 6850 2300
@@
 $EndComp
 $Comp
-L AZ1117-3.3 U3
+L smart-psu-rescue:AZ1117-3.3 U3
 U 1 1 5ACA8A4E
 P 5450 3550
@@
 $EndComp
 Wire Wire Line
-	4450 3550 4850 3550
-Wire Wire Line
-	2950 3550 3250 3550
-$Comp
-L GND #PWR12
+	4450 3550 4800 3550
+Wire Wire Line
+	2950 3550 3200 3550
+$Comp
+L power:GND #PWR12
 U 1 1 5ACA9DF6
 P 5450 4050
@@
 $EndComp
 $Comp
-L CP1_Small C3
+L Device:CP1_Small C3
 U 1 1 5A36723B
 P 5100 3900
@@
 $EndComp
 Wire Wire Line
-	5750 3550 6050 3550
+	5750 3550 5800 3550
 Wire Wire Line
 	5450 4050 5450 3850
@@
 	5100 3800 5100 3550
 Wire Wire Line
-	5050 3550 5150 3550
+	5050 3550 5100 3550
 Connection ~ 5100 3550
 Wire Wire Line
@@
 	8450 3950 8050 3950
 $Comp
-L Q_PMOS_GDS Q1
+L Device:Q_PMOS_GDS Q1
 U 1 1 5ACD007E
 P 7100 2200
@@
 	6550 2100 6600 2100
 Wire Wire Line
-	6800 2100 6900 2100
+	6800 2100 6850 2100
 Wire Wire Line
 	6850 2200 6850 2100
 Connection ~ 6850 2100
 $Comp
-L Q_NPN_BEC Q2
+L Device:Q_NPN_BEC Q2
 U 1 1 5ACD0E46
 P 7000 2700
@@
 	6850 2450 7100 2450
 Wire Wire Line
-	7100 2400 7100 2500
+	7100 2400 7100 2450
 Connection ~ 7100 2450
 $Comp
-L GND #PWR17
+L power:GND #PWR17
 U 1 1 5ACD1357
 P 7100 2950
@@
 Connection ~ 7500 2100
 $Comp
-L SW_DIP_x02 SW1
+L smart-psu-rescue:SW_DIP_x02 SW1
 U 1 1 5ACD3525
 P 8900 4800
@@
 $EndComp
 $Comp
-L GND #PWR20
+L power:GND #PWR20
 U 1 1 5ACD42F7
 P 9300 4900
@@
 	9200 4700 9300 4700
 Wire Wire Line
-	9300 4700 9300 4900
+	9300 4700 9300 4800
 Wire Wire Line
 	9200 4800 9300 4800
@@
 ~HB
 $Comp
-L Conn_01x05 J2
+L smart-psu-rescue:Conn_01x05 J2
 U 1 1 5ADDF8EA
 P 9250 3750
@@
 ~HB
 Wire Wire Line
-	7300 2100 7750 2100
-$Comp
-L R_Small R?
+	7300 2100 7500 2100
+$Comp
+L Device:R_Small R?
 U 1 1 5AFA8DEA
 P 6650 2700
@@
 Wire Wire Line
 	6750 2700 6800 2700
+Wire Wire Line
+	5800 3550 5800 3800
+Wire Wire Line
+	5800 3550 6050 3550
+Wire Wire Line
+	4500 3750 4550 3750
+Wire Wire Line
+	4800 3750 4800 3800
+Wire Wire Line
+	4800 3550 4800 3750
+Wire Wire Line
+	4800 3550 4850 3550
+Wire Wire Line
+	3200 3550 3250 3550
+Wire Wire Line
+	5100 3550 5150 3550
+Wire Wire Line
+	6850 2100 6900 2100
+Wire Wire Line
+	7100 2450 7100 2500
+Wire Wire Line
+	7500 2100 7750 2100
+Wire Wire Line
+	9300 4800 9300 4900
 $EndSCHEMATC

Commit message: Adding AC recovery configuration pin.
Connections:
- net labels added: DELAY, ~ACR
- net labels removed: DELAY1, DELAY2
Changed lines of the file:
@@
 LOAD
 Text Label 8450 3950 2    44   ~ 0
-DELAY1
+DELAY
 $Comp
 L Device:R_Small R2
@@
 FAULT
 Text Label 8300 4700 0    44   ~ 0
-DELAY1
+DELAY
 Text Label 8300 4800 0    44   ~ 0
-DELAY2
+~ACR
 Wire Wire Line
 	8750 3750 9050 3750
@@
 Connection ~ 5100 3550
 Wire Wire Line
-	8050 3550 8450 3550
-Wire Wire Line
 	8050 3650 8450 3650
 Wire Wire Line
@@
 Connection ~ 9300 4800
 Text Label 8450 4050 2    44   ~ 0
-DELAY2
+~ACR
 Wire Wire Line
 	8050 4050 8450 4050
@@
 Wire Wire Line
 	9300 4800 9300 4900
+Wire Wire Line
+	8050 3550 8450 3550
 $EndSCHEMATC

Commit message: Accidentaly delete rescue-lib
Parts:
- removed D1: 1N5824, Diodes_THT:D_DO-201AD_P12.70mm_Horizontal, symbol smart-psu-rescue:D_Schottky_Small_ALT
- removed D2: BAT54W, Diodes_SMD:D_1206, symbol smart-psu-rescue:D_Schottky_Small_ALT
- removed J1: 12V, Connectors_Terminal_Blocks:TerminalBlock_4UCON_19963_02x3.5mm_Straight, symbol smart-psu-rescue:Screw_Terminal_1x02
- removed J2: Conn_01x05, symbol smart-psu-rescue:Conn_01x05
- removed SW1: SW_DIP_x02, Buttons_Switches_THT:SW_DIP_x2_Slide, symbol smart-psu-rescue:SW_DIP_x02
- removed U1: LM2596, TO_SOT_Packages_SMD:TO-263-5_TabPin6, symbol smart-psu-rescue:LM2596
- removed U2: ATTINY13-20SSU, Housings_SOIC:SOIC-8_3.9x4.9mm_Pitch1.27mm, symbol smart-psu-rescue:ATTINY13-20SSU
- removed U3: AZ1117-3.3, Diodes_SMD:D_SOD-123, symbol smart-psu-rescue:AZ1117-3.3
- added D1: 1N5824, symbol Device:D_Small_ALT
- added D2: BAT54W, symbol Device:D_ALT
- added J1: 9-12V, symbol Connector_Generic:Conn_01x02
- added J2: HEADER, symbol Connector_Generic:Conn_01x05
- added SW1: SW_DIP_x02, symbol Switch:SW_DIP_x02
- added U1: LM2596S-5, Package_TO_SOT_SMD:TO-263-5_TabPin3, symbol Regulator_Switching:LM2596S-5
- added U2: AP1117-33, Package_TO_SOT_SMD:SOT-223-3_TabPin2, symbol Regulator_Linear:AP1117-33
- added U3: ATtiny13A-PU, Package_DIP:DIP-8_W7.62mm, symbol MCU_Microchip_ATtiny:ATtiny13A-PU
- gave numbers to parts that had none: 1
- renumbered Q2 to Q1, Q1 to Q2, R3 to R2, R2 to R3
Connections:
- net labels added: PWR
- wire segments 69 -> 68
Other:
- moved on the sheet: D3, F1, Q1, Q2, R1, R2, R3

Commit message: Update schematic
Parts:
- removed D1: 1N5824, symbol Device:D_Small_ALT
- removed D2: BAT54W, symbol Device:D_ALT
- removed J2: HEADER, symbol Connector_Generic:Conn_01x05
- added D1: 1N5824, symbol Device:D_Schottky_Small_ALT
- added D?: BAT54W, symbol Device:D_Schottky_Small_ALT
- added J2, J3: Conn_01x03, symbol Connector_Generic:Conn_01x03
- J1: value 9-12V -> DC-IN
- R1, R2, R3: footprint (none) -> Resistor_SMD:R_1206_3216Metric_Pad1.42x1.75mm_HandSolder
Connections:
- net labels added: DLY, FLT, GPIO, PWR_BT, PWR_SW, ~PWR
- net labels removed: +5V, DELAY, FAULT, PWR, VCC, ~BUTTON, ~HB, ~PWRON
- wire segments 68 -> 71
Other:
- note added: "ACR = AC RECOVERY\nPWR_BT = POWER SWITCH\nFLT = FAULT LED\nDLY = POWEROFF DELAY\nHBT = HEARTBEAT SIGNAL"
- moved on the sheet: C1, C2, C3, C4, D3, F1, J1, L1, Q1, Q2, R1, R2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

Commit message: Update schematic
Parts:
- removed D3: PWR, symbol Device:LED_Small_ALT
- removed J1: DC-IN, symbol Connector_Generic:Conn_01x02
- removed J2, J3: Conn_01x03, symbol Connector_Generic:Conn_01x03
- removed Q1: TUP, symbol Device:Q_NPN_BEC
- removed Q2: P2003ED, symbol Device:Q_PMOS_GDS
- removed U3: ATtiny13A-PU, Package_DIP:DIP-8_W7.62mm, symbol MCU_Microchip_ATtiny:ATtiny13A-PU
- added C4: 100n, Capacitor_SMD:C_1206_3216Metric_Pad1.33x1.80mm_HandSolder, symbol Device:C_Small
- added J1: DC-IN, TerminalBlock_MetzConnect:TerminalBlock_MetzConnect_Type055_RT01502HDWU_1x02_P5.00mm_Horizontal, symbol Connector:Screw_Terminal_01x02
- added J2: LOAD, TerminalBlock_MetzConnect:TerminalBlock_MetzConnect_Type055_RT01502HDWU_1x02_P5.00mm_Horizontal, symbol Connector:Screw_Terminal_01x02
- added J3: frontpanel, Connector_PinHeader_2.54mm:PinHeader_1x09_P2.54mm_Vertical, symbol Connector_Generic:Conn_01x09
- added L2: 22uH, Inductor_THT:L_Toroid_Vertical_L21.6mm_W11.4mm_P7.62mm_Pulse_KM-3, symbol Device:L_Small
- added Q1: MMBT3904, Package_TO_SOT_SMD:SOT-23, symbol Transistor_BJT:MMBT3904
- added Q2: P2003EVG, Package_SO:SOIC-8_3.9x4.9mm_P1.27mm, symbol Transistor_FET:P2003EVG
- added U3: ATtiny13-20SSU, Package_SO:SOIC-8_3.9x4.9mm_P1.27mm, symbol MCU_Microchip_ATtiny:ATtiny13-20SSU
- C1: footprint Capacitors_THT:CP_Radial_D10.0mm_P5.00mm_P7.50mm -> Capacitor_THT:C_Radial_D10.0mm_H20.0mm_P5.00mm
- C2: footprint Capacitors_THT:CP_Radial_D8.0mm_P3.50mm -> Capacitor_THT:CP_Radial_D8.0mm_P2.50mm
- C3: value 10u -> 100u; footprint Capacitors_THT:CP_Radial_D7.5mm_P2.50mm -> Capacitor_THT:CP_Radial_D5.0mm_P2.50mm
- C5: renamed from C4; footprint Capacitors_SMD:C_1206_HandSoldering -> Capacitor_SMD:C_1206_3216Metric_Pad1.33x1.80mm_HandSolder
- D1: footprint (none) -> Diode_THT:D_A-405_P12.70mm_Horizontal
- D2: renamed from D?; footprint (none) -> Diode_SMD:D_1206_3216Metric_Pad1.42x1.75mm_HandSolder
- F1: footprint SMD_Packages:SMD-1206_Pol -> Fuse:Fuse_1206_3216Metric_Pad1.42x1.75mm_HandSolder
- L1: footprint Choke_Toroid_ThroughHole:Choke_Toroid_6,5x13mm_Vertical -> Inductor_THT:L_Toroid_Vertical_L21.6mm_W11.4mm_P7.62mm_Pulse_KM-3
- R1: renamed from R2; footprint Resistor_SMD:R_1206_3216Metric_Pad1.42x1.75mm_HandSolder -> Resistor_SMD:R_1206_3216Metric_Pad1.30x1.75mm_HandSolder
- R2: renamed from R1; footprint Resistor_SMD:R_1206_3216Metric_Pad1.42x1.75mm_HandSolder -> Resistor_SMD:R_1206_3216Metric_Pad1.30x1.75mm_HandSolder
- R3: footprint Resistor_SMD:R_1206_3216Metric_Pad1.42x1.75mm_HandSolder -> Resistor_SMD:R_1206_3216Metric_Pad1.30x1.75mm_HandSolder
- SW1: footprint (none) -> Button_Switch_THT:SW_DIP_SPSTx02_Slide_9.78x7.26mm_W7.62mm_P2.54mm
Connections:
- net DLY: now also U3.3 (PB4)
- net GND: now also C4.2, J1.2 (Pin_2), J2.2 (Pin_2), J3.3 (Pin_3), J3.5 (Pin_5), J3.8 (Pin_8), J3.9 (Pin_9), Q1.2 (E), U3.4 (GND)
- net GPIO: now also J3.4 (Pin_4), U3.5 (PB0)
- net LOAD: now also J2.1 (Pin_1), J3.6 (Pin_6), J3.7 (Pin_7), Q2.5 (D), Q2.6 (D), Q2.7 (D), Q2.8 (D); no longer R3.2
- net PWR_SW: now also J3.2 (Pin_2), U3.6 (PB1)
- net ~ACR: now also U3.1 (~RESET~/PB5)
- net ~PWR: now also U3.7 (PB2)
- net at C2.1, L1.2, U1.4 (FB): now also L2.2; no longer D2.2 (A), F1.1
- net at F1.2: now also C1.1, U1.1 (VIN); no longer R1.2
- net LED: now reaches R3.1
- net LED: now also U3.2 (PB3)
- net at R1.1: now also Q1.3 (C), Q2.4 (G)
- net at R2.2: now also Q1.1 (B)
- net at C5.1, U2.2 (VO): now also U3.8 (VCC)
- net at D2.1 (K), U2.3 (VI): no longer C3.1
- new net: F1.1, J1.1 (Pin_1)
- new net: J3.1 (Pin_1), R3.2
- new net: C3.1, C4.1, D2.2 (A), L2.1, Q2.1 (S), Q2.2 (S), Q2.3 (S), R1.2
Other:
- note added: "= AC RECOVERY\n= POWER SWITCH\n= ON/ALARM LED\n= POWEROFF DELAY\n= TO SBC GPIO"
- note added: "ACR \nPWR_SW \nLED \nDLY\nGPIO"
- note removed: "ACR = AC RECOVERY\nPWR_BT = POWER SWITCH\nFLT = FAULT LED\nDLY = POWEROFF DELAY\nHBT = HEARTBEAT SIGNAL"
- moved on the sheet: C1, C2, C3, D1, D2, F1, L1, R1, R3, U1
